Commit message: Create camera link and joint

File: my_robot/urdf/my_robot.xacro (robot description, xacro)
@@ -1,4 +1,35 @@
 <?xml version='1.0'?>
 <robot name="my_robot" xmlns:xacro="http://www.ros.org/wiki/xacro">
+  <link name="camera">
+    <inertial>
+      <mass value="0.1"/>
+      <origin xyz="0 0 0" rpy="0 0 0 "/>
+      <inertia
+          ixx="1e-6" ixy="0" ixz="0"
+          iyy="1e-6" iyz="0"
+          izz="1e-6"
+      />
+    </inertial>
+    <collision name='collision'>
+      <origin xyz="0 0 0" rpy=" 0 0 0"/>
+      <geometry>
+        <box size=".05 .05 .05"/>
+      </geometry>
+    </collision>
+    <visual name='camera_visual'>
+      <origin xyz="0 0 0" rpy=" 0 0 0"/>
+      <geometry>
+         <box size=".05 .05 .05"/>
+      </geometry>
+    </visual>
+  </link>
+  <joint type="fixed" name="camera_joint">
+    <origin xyz="0.2 0 0" rpy="0 0 0"/>
+    <child link="camera"/>
+    <parent link="chassis"/>
+    <axis xyz="0 1 0" rpy="0 0 0"/>
+    <limit effort="10000" velocity="1000"/>
+    <dynamics damping="1.0" friction="1.0"/>
+  </joint>
   <link name="robot_footprint"></link>
   <joint name="robot_footprint_joint" type="fixed">
@@ -109,5 +140,5 @@
     </visual>
   </link>
-   <joint type="continuous" name="left_wheel_hinge">
+  <joint type="continuous" name="left_wheel_hinge">
     <origin xyz="0 0.15 0" rpy="0 0 0"/>
     <child link="left_wheel"/>

Commit message: Update the robot's newest features

File: my_robot/urdf/my_robot.xacro (robot description, xacro)
@@ -1,13 +1,54 @@
 <?xml version='1.0'?>
 <robot name="my_robot" xmlns:xacro="http://www.ros.org/wiki/xacro">
-  <link name="camera">
+  <link name="robot_footprint"></link>
+  <joint name="robot_footprint_joint" type="fixed">
+    <origin xyz="0 0 0" rpy="0 0 0" />
+    <parent link="robot_footprint"/>
+    <child link="chassis" />
+  </joint>
+  <joint name="hokuyo_joint" type="fixed">
+    <origin xyz="0.15 0 0.1" rpy="0 0 0"/>
+    <child link="hokuyo"/>
+    <parent link="chassis"/>
+    <axis xyz="0 1 0" rpy="0 0 0"/>
+  </joint>
+  <link name='hokuyo'>
+    <inertial>
+      <mass value="1e-5"/>
+      <origin xyz="0 0 0" rpy="0 0 0 "/>
+       <inertia
+          ixx="1e-6" ixy="0" ixz="0"
+          iyy="1e-6" iyz="0"
+          izz="1e-6"
+       />
+    </inertial>
+    <collision name='collision'>
+      <origin xyz="0 0 0" rpy=" 0 0 0"/>
+      <geometry>
+        <box size="0.1 0.1 0.1"/>
+      </geometry>
+    </collision>
+    <visual name='hokuyo_visual'>
+      <origin xyz="0 0 0" rpy=" 0 0 0"/>
+      <geometry>
+        <mesh filename="package://my_robot/meshes/hokuyo.dae"/>
+      </geometry>
+    </visual>
+  </link>
+  <joint name="camera_joint" type="fixed">
+    <origin xyz="0.3 0 0" rpy="0 0 0"/>
+    <child link="camera"/>
+    <parent link="chassis"/>
+    <axis xyz="0 1 0" rpy="0 0 0"/>
+  </joint>
+  <link name='camera'>
     <inertial>
       <mass value="0.1"/>
       <origin xyz="0 0 0" rpy="0 0 0 "/>
-      <inertia
+       <inertia
           ixx="1e-6" ixy="0" ixz="0"
           iyy="1e-6" iyz="0"
           izz="1e-6"
-      />
+       />
     </inertial>
     <collision name='collision'>
@@ -24,20 +65,4 @@
     </visual>
   </link>
-  <joint type="fixed" name="camera_joint">
-    <origin xyz="0.2 0 0" rpy="0 0 0"/>
-    <child link="camera"/>
-    <parent link="chassis"/>
-    <axis xyz="0 1 0" rpy="0 0 0"/>
-    <limit effort="10000" velocity="1000"/>
-    <dynamics damping="1.0" friction="1.0"/>
-  </joint>
-=======
->>>>>>> bd0ab9d1d7ee115b83019bf9c6dd23eab5bfe4af
-  <link name="robot_footprint"></link>
-  <joint name="robot_footprint_joint" type="fixed">
-    <origin xyz="0 0 0" rpy="0 0 0" />
-    <parent link="robot_footprint"/>
-    <child link="chassis" />
-  </joint>
   <link name='chassis'>
     <pose>0 0 0.1 0 0 0</pose>
@@ -88,4 +113,12 @@
     </visual>
   </link>
+  <joint name="right_wheel_hinge" type="continuous">
+    <origin xyz="0 -0.15 0" rpy="0 0 0"/>
+    <child link="right_wheel"/>
+    <parent link="chassis"/>
+    <axis xyz="0 1 0" rpy="0 0 0"/>
+    <limit effort="10000" velocity="1000"/>
+    <dynamics damping="1.0" friction="1.0"/>
+  </joint>
   <link name="right_wheel">
     <inertial>
@@ -98,6 +131,4 @@
       />
     </inertial>
-<<<<<<< HEAD
-=======
     <collision name='collision'>
       <origin xyz="0 0 0" rpy=" 0 1.5707 1.5707"/>
@@ -113,7 +144,7 @@
     </visual>
   </link>
-  <joint type="continuous" name="right_wheel_hinge">
-    <origin xyz="0 -0.15 0" rpy="0 0 0"/>
-    <child link="right_wheel"/>
+  <joint name="left_wheel_hinge" type="continuous">
+    <origin xyz="0 0.15 0" rpy="0 0 0"/>
+    <child link="left_wheel"/>
     <parent link="chassis"/>
     <axis xyz="0 1 0" rpy="0 0 0"/>
@@ -144,64 +175,3 @@
     </visual>
   </link>
-   <joint type="continuous" name="left_wheel_hinge">
-    <origin xyz="0 0.15 0" rpy="0 0 0"/>
-    <child link="left_wheel"/>
-    <parent link="chassis"/>
-    <axis xyz="0 1 0" rpy="0 0 0"/>
-    <limit effort="10000" velocity="1000"/>
-    <dynamics damping="1.0" friction="1.0"/>
-  </joint>
->>>>>>> bd0ab9d1d7ee115b83019bf9c6dd23eab5bfe4af
-    <collision name='collision'>
-      <origin xyz="0 0 0" rpy=" 0 1.5707 1.5707"/>
-      <geometry>
-        <cylinder radius="0.1" length="0.05"/>
-      </geometry>
-    </collision>
-    <visual name='right_wheel_visual'>
-      <origin xyz="0 0 0" rpy=" 0 1.5707 1.5707"/>
-      <geometry>
-         <cylinder radius="0.1" length="0.05"/>
-      </geometry>
-    </visual>
-  </link>
-  <joint type="continuous" name="right_wheel_hinge">
-    <origin xyz="0 -0.15 0" rpy="0 0 0"/>
-    <child link="right_wheel"/>
-    <parent link="chassis"/>
-    <axis xyz="0 1 0" rpy="0 0 0"/>
-    <limit effort="10000" velocity="1000"/>
-    <dynamics damping="1.0" friction="1.0"/>
-  </joint>
-  <link name="left_wheel">
-    <inertial>
-      <mass value="5"/>
-      <origin xyz="0 0 0" rpy=" 0 1.5707 1.5707"/>
-      <inertia
-          ixx="0.1" ixy="0" ixz="0"
-          iyy="0.1" iyz="0"
-          izz="0.1"
-      />
-    </inertial>
-    <collision name='collision'>
-      <origin xyz="0 0 0" rpy=" 0 1.5707 1.5707"/>
-      <geometry>
-        <cylinder radius="0.1" length="0.05"/>
-      </geometry>
-    </collision>
-    <visual name='left_wheel_visual'>
-      <origin xyz="0 0 0" rpy=" 0 1.5707 1.5707"/>
-      <geometry>
-         <cylinder radius="0.1" length="0.05"/>
-      </geometry>
-    </visual>
-  </link>
-  <joint type="continuous" name="left_wheel_hinge">
-    <origin xyz="0 0.15 0" rpy="0 0 0"/>
-    <child link="left_wheel"/>
-    <parent link="chassis"/>
-    <axis xyz="0 1 0" rpy="0 0 0"/>
-    <limit effort="10000" velocity="1000"/>
-    <dynamics damping="1.0" friction="1.0"/>
-  </joint>
 </robot>

Commit message: Update the robot's appearance (colors)

File: my_robot/urdf/my_robot.xacro (robot description, xacro)
@@ -176,3 +176,15 @@
     </visual>
   </link>
+  <gazebo reference="chassis">
+    <material>Gazebo/Green</material>
+  </gazebo>
+  <gazebo reference="left_wheel">
+    <material>Gazebo/Yellow</material>
+  </gazebo>
+  <gazebo reference="right_wheel">
+    <material>Gazebo/Yellow</material>
+  </gazebo>
+  <gazebo reference="camera">
+    <material>Gazebo/Blue</material>
+  </gazebo>
 </robot>

Commit message: Create the ball_chaser pkg

File: my_robot/urdf/my_robot.xacro (robot description, xacro)
@@ -177,14 +177,14 @@
   </link>
   <gazebo reference="chassis">
+    <material>Gazebo/Blue</material>
+  </gazebo>
+  <gazebo reference="left_wheel">
     <material>Gazebo/Green</material>
   </gazebo>
-  <gazebo reference="left_wheel">
-    <material>Gazebo/Yellow</material>
-  </gazebo>
   <gazebo reference="right_wheel">
-    <material>Gazebo/Yellow</material>
+    <material>Gazebo/Green</material>
   </gazebo>
   <gazebo reference="camera">
-    <material>Gazebo/Blue</material>
+    <material>Gazebo/Red</material>
   </gazebo>
 </robot>
